File: schematic/WirelessCTSensors.kicad_pcb (KiCad board)
At the start: 2 copper layers, 38.1 x 41.9 mm, 28 parts, among them IC1 ATTINY85-S, J1 Clamp2, J2 Clamp3, J3 Clamp1, P1 Power Connector, P2 CONN_01X02, SW1 RESET, SW2 RESCUE_MODE, U1 LM1117 3.3, U2 ESP-01

Commit message: Update schematic with KiCad 5.1.4
Parts:
- IC1: value ATTINY85-S -> ATtiny85-20SU
- P1: footprint Connect:bornier2 -> Terminal_Blocks:TerminalBlock_bornier-2_P5.08mm
- P2: value CONN_01X02 -> Serial Out
- U1: value LM1117 3.3 -> AP1117-33
- moved P1 2.54 mm to (156.2, 87.6)
Changed lines of the file:
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@@
-(kicad_pcb (version 4) (host pcbnew 4.0.6)
+(kicad_pcb (version 20171130) (host pcbnew "(5.1.4)-1")
   (general
-    (links 67)
-    (no_connects 0)
-    (area 126.115 72.865 179.935 129.025001)
     (thickness 1.6)
     (drawings 14)
@@
     (zone_45_only no)
     (trace_min 0.1524)
-    (segment_width 0.2)
-    (edge_width 0.15)
     (via_size 0.6858)
     (via_drill 0.3302)
@@
     (uvia_min_size 0)
     (uvia_min_drill 0)
+    (edge_width 0.15)
+    (segment_width 0.2)
     (pcb_text_width 0.3)
     (pcb_text_size 1.5 1.5)
@@
       (layerselection 0x010f0_80000001)
       (usegerberextensions true)
+      (usegerberattributes false)
+      (usegerberadvancedattributes false)
+      (creategerberjobfile false)
       (excludeedgelayer true)
       (linewidth 0.100000)
@@
       (hpglpennumber 1)
       (hpglpenspeed 20)
-      (hpglpendiameter 15)
-      (hpglpenoverlay 2)
+      (hpglpendiameter 15.000000)
       (psnegative false)
       (psa4output false)
@@
       (drillshape 0)
       (scaleselection 1)
-      (outputdirectory gerber))
+      (outputdirectory "gerber"))
   )
   (net 0 "")
@@
       (effects (font (size 1 1) (thickness 0.15)))
     )
-    (fp_text value "LM1117 3.3" (at 0 0.762 90) (layer F.Fab)
+    (fp_text value AP1117-33 (at 0 0.762 90) (layer F.Fab)
       (effects (font (size 1 1) (thickness 0.15)))
     )
@@
     (descr "8-lead dip package, row spacing 7.62 mm (300 mils), longer pads")
     (tags "dil dip 2.54 300")
-    (fp_text reference IC1 (at 2.413 11.049 360) (layer F.SilkS)
-      (effects (font (size 1 1) (thickness 0.15)))
-    )
-    (fp_text value ATTINY85-S (at 0 -3.72 270) (layer F.Fab)
+    (fp_text reference IC1 (at 2.413 11.049) (layer F.SilkS)
+      (effects (font (size 1 1) (thickness 0.15)))
+    )
+    (fp_text value ATtiny85-20SU (at 0 -3.72 270) (layer F.Fab)
       (effects (font (size 1 1) (thickness 0.15)))
     )
@@
       (net 6 VCC))
     (model Housings_DIP.3dshapes/DIP-8_W7.62mm_LongPads.wrl
-      (at (xyz 0 0 0))
-      (scale (xyz 1 1 1))
-      (rotate (xyz 0 0 0))
-    )
-  )
-  (module Connect:bornier2 placed (layer F.Cu)
-    (at 158.75 87.63)
-    (descr "Bornier d'alimentation 2 pins")
-    (tags DEV)
-    (fp_text reference P1 (at 0 -2.413) (layer F.SilkS)
-      (effects (font (size 1 1) (thickness 0.15)))
-    )
-    (fp_text value "Power Connector" (at 0 5.08) (layer F.Fab)
-      (effects (font (size 1 1) (thickness 0.15)))
-    )
-    (fp_line (start 5.08 2.54) (end -5.08 2.54) (layer F.SilkS) (width 0.15))
-    (fp_line (start 5.08 3.81) (end 5.08 -3.81) (layer F.SilkS) (width 0.15))
-    (fp_line (start 5.08 -3.81) (end -5.08 -3.81) (layer F.SilkS) (width 0.15))
-    (fp_line (start -5.08 -3.81) (end -5.08 3.81) (layer F.SilkS) (width 0.15))
-    (fp_line (start -5.08 3.81) (end 5.08 3.81) (layer F.SilkS) (width 0.15))
-    (pad 1 thru_hole rect (at -2.54 0) (size 2.54 2.54) (drill 1.524) (layers *.Cu *.Mask F.SilkS)
-      (net 2 GND))
-    (pad 2 thru_hole circle (at 2.54 0) (size 2.54 2.54) (drill 1.524) (layers *.Cu *.Mask F.SilkS)
-      (net 6 VCC))
-    (model Connect.3dshapes/bornier2.wrl
       (at (xyz 0 0 0))
       (scale (xyz 1 1 1))
@@
     (tags "Tantal Cap. , Size B, EIA-3528, Hand Soldering,")
     (attr smd)
-    (fp_text reference C1 (at -4.826 0 360) (layer F.SilkS)
+    (fp_text reference C1 (at -4.826 0) (layer F.SilkS)
       (effects (font (size 1 1) (thickness 0.15)))
     )
@@
     (tags "Tantal Cap. , Size A, EIA-3216, Hand Soldering,")
     (attr smd)
-    (fp_text reference C5 (at -4.699 -0.127 360) (layer B.SilkS)
+    (fp_text reference C5 (at -4.699 -0.127) (layer B.SilkS)
       (effects (font (size 1 1) (thickness 0.15)) (justify mirror))
     )
@@
       (effects (font (size 1 1) (thickness 0.15)))
     )
-    (fp_text value CONN_01X02 (at 0 4.93 180) (layer F.Fab)
+    (fp_text value "Serial Out" (at 0 4.93 180) (layer F.Fab)
       (effects (font (size 1 1) (thickness 0.15)))
     )
@@
       (net 14 "Net-(P2-Pad2)"))
     (model Pin_Headers.3dshapes/Pin_Header_Straight_1x02_Pitch2.54mm.wrl
-      (at (xyz 0 -0.05 0))
+      (offset (xyz 0 -1.269999980926514 0))
       (scale (xyz 1 1 1))
       (rotate (xyz 0 0 90))
@@
       (scale (xyz 1 1 1))
       (rotate (xyz 0 0 0))
+    )
+  )
+  (module Terminal_Blocks:TerminalBlock_bornier-2_P5.08mm (layer F.Cu)
+    (at 156.21 87.63)
+    (descr "simple 2-pin terminal block, pitch 5.08mm, revamped version of bornier2")
+    (tags "terminal block bornier2")
+    (fp_text reference P1 (at 2.54 -5.08) (layer F.SilkS)
+      (effects (font (size 1 1) (thickness 0.15)))
+    )
+    (fp_text value "Power Connector" (at 2.54 5.08) (layer F.Fab)
+      (effects (font (size 1 1) (thickness 0.15)))
+    )
+    (fp_line (start 7.79 4) (end -2.71 4) (layer F.CrtYd) (width 0.05))
+    (fp_line (start 7.79 4) (end 7.79 -4) (layer F.CrtYd) (width 0.05))
+    (fp_line (start -2.71 -4) (end -2.71 4) (layer F.CrtYd) (width 0.05))
+    (fp_line (start -2.71 -4) (end 7.79 -4) (layer F.CrtYd) (width 0.05))
+    (fp_line (start -2.54 3.81) (end 7.62 3.81) (layer F.SilkS) (width 0.12))
+    (fp_line (start -2.54 -3.81) (end -2.54 3.81) (layer F.SilkS) (width 0.12))
+    (fp_line (start 7.62 -3.81) (end -2.54 -3.81) (layer F.SilkS) (width 0.12))
+    (fp_line (start 7.62 3.81) (end 7.62 -3.81) (layer F.SilkS) (width 0.12))
+    (fp_line (start 7.62 2.54) (end -2.54 2.54) (layer F.SilkS) (width 0.12))
+    (fp_line (start 7.54 -3.75) (end -2.46 -3.75) (layer F.Fab) (width 0.1))
+    (fp_line (start 7.54 3.75) (end 7.54 -3.75) (layer F.Fab) (width 0.1))
+    (fp_line (start -2.46 3.75) (end 7.54 3.75) (layer F.Fab) (width 0.1))
+    (fp_line (start -2.46 -3.75) (end -2.46 3.75) (layer F.Fab) (width 0.1))
+    (fp_line (start -2.41 2.55) (end 7.49 2.55) (layer F.Fab) (width 0.1))
+    (fp_text user %R (at 2.54 0) (layer F.Fab)
+      (effects (font (size 1 1) (thickness 0.15)))
+    )
+    (pad 2 thru_hole circle (at 5.08 0) (size 3 3) (drill 1.52) (layers *.Cu *.Mask)
+      (net 6 VCC))
+    (pad 1 thru_hole rect (at 0 0) (size 3 3) (drill 1.52) (layers *.Cu *.Mask)
+      (net 2 GND))
+    (model ${KISYS3DMOD}/Terminal_Blocks.3dshapes/TerminalBlock_bornier-2_P5.08mm.wrl
+      (offset (xyz 2.539999961853027 0 0))
+      (scale (xyz 1 1 1))
+      (rotate (xyz 0 0 0))
