File: schematic/WirelessCTSensors.sch (KiCad schematic (older format))
At the start: 28 parts, among them IC1 ATTINY85-S, J1 Clamp2, J2 Clamp3, J3 Clamp1, P1 Power Connector, P2 CONN_01X02, SW1 RESET, SW2 RESCUE_MODE, U1 LM1117 3.3, U2 ESP-01

Commit message: Update schematic with KiCad 5.1.4
Parts:
- removed IC1: ATTINY85-S, Housings_DIP:DIP-8_W7.62mm_LongPads, symbol ATTINY85-S
- removed P1: Power Connector, Connect:bornier2, symbol CONN_01X02
- removed P2: CONN_01X02, Pin_Headers:Pin_Header_Straight_1x02_Pitch2.54mm, symbol CONN_01X02
- removed SW1: RESET, Buttons_Switches_ThroughHole:SW_PUSH_6mm, symbol SW_PUSH
- removed SW2: RESCUE_MODE, Buttons_Switches_ThroughHole:SW_PUSH_6mm, symbol SW_PUSH
- removed U1: LM1117 3.3, TO_SOT_Packages_SMD:SOT-223, symbol AP1117D33
- added IC1: ATtiny85-20SU, Housings_DIP:DIP-8_W7.62mm_LongPads, symbol MCU_Microchip_ATtiny:ATtiny85-20SU
- added P1: Power Connector, Terminal_Blocks:TerminalBlock_bornier-2_P5.08mm, symbol Connector_Generic:Conn_01x02
- added P2: Serial Out, Pin_Headers:Pin_Header_Straight_1x02_Pitch2.54mm, symbol Connector_Generic:Conn_01x02
- added SW1: RESET, Buttons_Switches_ThroughHole:SW_PUSH_6mm, symbol Switch:SW_Push
- added SW2: RESCUE_MODE, Buttons_Switches_ThroughHole:SW_PUSH_6mm, symbol Switch:SW_Push
- added U1: AP1117-33, TO_SOT_Packages_SMD:SOT-223, symbol Regulator_Linear:AP1117-33
- C1, C5: symbol CP -> Device:CP
- C2, C3, C4: symbol C_Small -> Device:C_Small
- D1, D2, D3, D4, D5, D6: symbol D -> Device:D
- J1, J2, J3: symbol JACK_TRS_5PINS -> jack_trs_5pins:JACK_TRS_5PINS
- R1, R2, R3, R4, R5, R6, R7: symbol R -> Device:R
- U2: symbol ESP-01v090 -> ESP8266:ESP-01v090
Connections:
- net GND: now also IC1.4 (GND), P1.1 (Pin_1), P2.1 (Pin_1), SW1.2, SW2.2, U1.1 (GND)
- net VCC: now also IC1.8 (VCC), P1.2 (Pin_2), U1.3 (VI)
- net VCC2: now also U1.2 (VO)
- net at U2.1 (UTXD): now also P2.2 (Pin_2)
- net at U2.4 (GPIO2): now also SW2.1
- net at U2.5 (RST): now also SW1.1
- net at U2.8 (URXD): now also IC1.5 (AREF/PB0)
- net at R7.1: now also IC1.1 (~RESET~/PB5)
- net at D3.2 (A), D4.1 (K), J2.4 (TN)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: now also IC1.2 (XTAL1/PB3)
- net at D5.2 (A), D6.1 (K), J3.4 (TN)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: now also IC1.3 (XTAL2/PB4)
- net at D1.2 (A), D2.1 (K), J1.4 (TN)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: now also IC1.7 (PB2)

Commit message: Update schematic
Parts:
- C1: footprint Capacitors_Tantalum_SMD:TantalC_SizeB_EIA-3528_HandSoldering -> Capacitor_Tantalum_SMD:CP_EIA-3528-21_Kemet-B_Pad1.50x2.35mm_HandSolder
- C2, C3, C4: footprint Capacitors_SMD:C_0805_HandSoldering -> Capacitor_SMD:C_0805_2012Metric_Pad1.15x1.40mm_HandSolder
- C5: footprint Capacitors_Tantalum_SMD:TantalC_SizeA_EIA-3216_HandSoldering -> Capacitor_Tantalum_SMD:CP_EIA-3216-18_Kemet-A_Pad1.58x1.35mm_HandSolder
- D1, D2, D3, D4, D5, D6: footprint Clean Diode SMA:SMA_Handsoldering -> Diode_SMD:D_SMA_Handsoldering
- IC1: footprint Housings_DIP:DIP-8_W7.62mm_LongPads -> Package_DIP:DIP-8_W7.62mm_Socket_LongPads
- P1: footprint Terminal_Blocks:TerminalBlock_bornier-2_P5.08mm -> TerminalBlock:TerminalBlock_bornier-2_P5.08mm
- P2: footprint Pin_Headers:Pin_Header_Straight_1x02_Pitch2.54mm -> Connector_PinHeader_2.54mm:PinHeader_1x02_P2.54mm_Vertical
- R1, R2, R3, R4, R5, R6, R7: footprint Resistors_SMD:R_0805_HandSoldering -> Resistor_SMD:R_0805_2012Metric_Pad1.15x1.40mm_HandSolder
- SW1, SW2: footprint Buttons_Switches_ThroughHole:SW_PUSH_6mm -> Button_Switch_THT:SW_PUSH_6mm
- U1: footprint TO_SOT_Packages_SMD:SOT-223 -> Package_TO_SOT_SMD:SOT-223-3_TabPin2
Changed lines of the file:
@@
 EESchema Schematic File Version 4
-LIBS:WirelessCTSensors-cache
 EELAYER 30 0
 EELAYER END
@@
 F 0 "C2" H 2110 2670 50  0000 L CNN
 F 1 "10uF" H 2110 2520 50  0000 L CNN
-F 2 "Capacitors_SMD:C_0805_HandSoldering" H 2100 2600 50  0001 C CNN
+F 2 "Capacitor_SMD:C_0805_2012Metric_Pad1.15x1.40mm_HandSolder" H 2100 2600 50  0001 C CNN
 F 3 "" H 2100 2600 50  0000 C CNN
 	1    2100 2600
@@
 F 0 "R2" V 2430 2600 50  0000 C CNN
 F 1 "330K" V 2350 2600 50  0000 C CNN
-F 2 "Resistors_SMD:R_0805_HandSoldering" V 2280 2600 50  0001 C CNN
+F 2 "Resistor_SMD:R_0805_2012Metric_Pad1.15x1.40mm_HandSolder" V 2280 2600 50  0001 C CNN
 F 3 "" H 2350 2600 50  0000 C CNN
 	1    2350 2600
@@
 F 0 "R1" V 2430 2200 50  0000 C CNN
 F 1 "330K" V 2350 2200 50  0000 C CNN
-F 2 "Resistors_SMD:R_0805_HandSoldering" V 2280 2200 50  0001 C CNN
+F 2 "Resistor_SMD:R_0805_2012Metric_Pad1.15x1.40mm_HandSolder" V 2280 2200 50  0001 C CNN
 F 3 "" H 2350 2200 50  0000 C CNN
 	1    2350 2200
@@
 F 0 "C1" H 2525 1250 50  0000 L CNN
 F 1 "100uF" H 2525 1050 50  0000 L CNN
-F 2 "Capacitors_Tantalum_SMD:TantalC_SizeB_EIA-3528_HandSoldering" H 2538 1000 50  0001 C CNN
+F 2 "Capacitor_Tantalum_SMD:CP_EIA-3528-21_Kemet-B_Pad1.50x2.35mm_HandSolder" H 2538 1000 50  0001 C CNN
 F 3 "" H 2500 1150 50  0000 C CNN
 	1    2500 1150
@@
 F 0 "C3" H 2060 4020 50  0000 L CNN
 F 1 "10uF" H 2060 3870 50  0000 L CNN
-F 2 "Capacitors_SMD:C_0805_HandSoldering" H 2050 3950 50  0001 C CNN
+F 2 "Capacitor_SMD:C_0805_2012Metric_Pad1.15x1.40mm_HandSolder" H 2050 3950 50  0001 C CNN
 F 3 "" H 2050 3950 50  0000 C CNN
 	1    2050 3950
@@
 F 0 "R4" V 2380 3950 50  0000 C CNN
 F 1 "330K" V 2300 3950 50  0000 C CNN
-F 2 "Resistors_SMD:R_0805_HandSoldering" V 2230 3950 50  0001 C CNN
+F 2 "Resistor_SMD:R_0805_2012Metric_Pad1.15x1.40mm_HandSolder" V 2230 3950 50  0001 C CNN
 F 3 "" H 2300 3950 50  0000 C CNN
 	1    2300 3950
@@
 F 0 "R3" V 2380 3550 50  0000 C CNN
 F 1 "330K" V 2300 3550 50  0000 C CNN
-F 2 "Resistors_SMD:R_0805_HandSoldering" V 2230 3550 50  0001 C CNN
+F 2 "Resistor_SMD:R_0805_2012Metric_Pad1.15x1.40mm_HandSolder" V 2230 3550 50  0001 C CNN
 F 3 "" H 2300 3550 50  0000 C CNN
 	1    2300 3550
@@
 F 0 "C4" H 2060 5320 50  0000 L CNN
 F 1 "10uF" H 2060 5170 50  0000 L CNN
-F 2 "Capacitors_SMD:C_0805_HandSoldering" H 2050 5250 50  0001 C CNN
+F 2 "Capacitor_SMD:C_0805_2012Metric_Pad1.15x1.40mm_HandSolder" H 2050 5250 50  0001 C CNN
 F 3 "" H 2050 5250 50  0000 C CNN
 	1    2050 5250
@@
 F 0 "R6" V 2380 5250 50  0000 C CNN
 F 1 "330K" V 2300 5250 50  0000 C CNN
-F 2 "Resistors_SMD:R_0805_HandSoldering" V 2230 5250 50  0001 C CNN
+F 2 "Resistor_SMD:R_0805_2012Metric_Pad1.15x1.40mm_HandSolder" V 2230 5250 50  0001 C CNN
 F 3 "" H 2300 5250 50  0000 C CNN
 	1    2300 5250
@@
 F 0 "R5" V 2380 4850 50  0000 C CNN
 F 1 "330K" V 2300 4850 50  0000 C CNN
-F 2 "Resistors_SMD:R_0805_HandSoldering" V 2230 4850 50  0001 C CNN
+F 2 "Resistor_SMD:R_0805_2012Metric_Pad1.15x1.40mm_HandSolder" V 2230 4850 50  0001 C CNN
 F 3 "" H 2300 4850 50  0000 C CNN
 	1    2300 4850
@@
 F 0 "D5" H 2700 5650 50  0000 C CNN
 F 1 "1N4002" H 2700 5450 50  0000 C CNN
-F 2 "Clean Diode SMA:SMA_Handsoldering" H 2700 5550 50  0001 C CNN
+F 2 "Diode_SMD:D_SMA_Handsoldering" H 2700 5550 50  0001 C CNN
 F 3 "" H 2700 5550 50  0000 C CNN
 	1    2700 5550
@@
 F 0 "D6" H 2700 6050 50  0000 C CNN
 F 1 "1N4002" H 2700 5850 50  0000 C CNN
-F 2 "Clean Diode SMA:SMA_Handsoldering" H 2700 5950 50  0001 C CNN
+F 2 "Diode_SMD:D_SMA_Handsoldering" H 2700 5950 50  0001 C CNN
 F 3 "" H 2700 5950 50  0000 C CNN
 	1    2700 5950
@@
 F 0 "D4" H 2700 4700 50  0000 C CNN
 F 1 "1N4002" H 2700 4500 50  0000 C CNN
-F 2 "Clean Diode SMA:SMA_Handsoldering" H 2700 4600 50  0001 C CNN
+F 2 "Diode_SMD:D_SMA_Handsoldering" H 2700 4600 50  0001 C CNN
 F 3 "" H 2700 4600 50  0000 C CNN
 	1    2700 4600
@@
 F 0 "D3" H 2700 4300 50  0000 C CNN
 F 1 "1N4002" H 2700 4100 50  0000 C CNN
-F 2 "Clean Diode SMA:SMA_Handsoldering" H 2700 4200 50  0001 C CNN
+F 2 "Diode_SMD:D_SMA_Handsoldering" H 2700 4200 50  0001 C CNN
 F 3 "" H 2700 4200 50  0000 C CNN
 	1    2700 4200
@@
 F 0 "D2" H 2700 3400 50  0000 C CNN
 F 1 "1N4002" H 2700 3200 50  0000 C CNN
-F 2 "Clean Diode SMA:SMA_Handsoldering" H 2700 3300 50  0001 C CNN
+F 2 "Diode_SMD:D_SMA_Handsoldering" H 2700 3300 50  0001 C CNN
 F 3 "" H 2700 3300 50  0000 C CNN
 	1    2700 3300
@@
 F 0 "D1" H 2700 3000 50  0000 C CNN
 F 1 "1N4002" H 2700 2800 50  0000 C CNN
-F 2 "Clean Diode SMA:SMA_Handsoldering" H 2700 2900 50  0001 C CNN
+F 2 "Diode_SMD:D_SMA_Handsoldering" H 2700 2900 50  0001 C CNN
 F 3 "" H 2700 2900 50  0000 C CNN
 	1    2700 2900
@@
 F 0 "C5" H 1525 1300 50  0000 L CNN
 F 1 "10uF" H 1525 1100 50  0000 L CNN
-F 2 "Capacitors_Tantalum_SMD:TantalC_SizeA_EIA-3216_HandSoldering" H 1538 1050 50  0001 C CNN
+F 2 "Capacitor_Tantalum_SMD:CP_EIA-3216-18_Kemet-A_Pad1.58x1.35mm_HandSolder" H 1538 1050 50  0001 C CNN
 F 3 "" H 1500 1200 50  0000 C CNN
 	1    1500 1200
@@
 F 0 "R7" V 3530 4450 50  0000 C CNN
 F 1 "10K" V 3450 4450 50  0000 C CNN
-F 2 "Resistors_SMD:R_0805_HandSoldering" V 3380 4450 50  0001 C CNN
+F 2 "Resistor_SMD:R_0805_2012Metric_Pad1.15x1.40mm_HandSolder" V 3380 4450 50  0001 C CNN
 F 3 "" H 3450 4450 50  0000 C CNN
 	1    3450 4450
@@
 F 0 "U1" H 1950 1242 50  0000 C CNN
 F 1 "AP1117-33" H 1950 1151 50  0000 C CNN
-F 2 "TO_SOT_Packages_SMD:SOT-223" H 1950 1200 50  0001 C CNN
+F 2 "Package_TO_SOT_SMD:SOT-223-3_TabPin2" H 1950 1200 50  0001 C CNN
 F 3 "http://www.diodes.com/datasheets/AP1117.pdf" H 2050 750 50  0001 C CNN
 	1    1950 1000
@@
 F 0 "IC1" H 3620 3996 50  0000 R CNN
 F 1 "ATtiny85-20SU" H 3620 3905 50  0000 R CNN
-F 2 "Housings_DIP:DIP-8_W7.62mm_LongPads" H 4150 3950 50  0001 C CIN
+F 2 "Package_DIP:DIP-8_W7.62mm_Socket_LongPads" H 4150 3950 50  0001 C CIN
 F 3 "http://ww1.microchip.com/downloads/en/DeviceDoc/atmel-2586-avr-8-bit-microcontroller-attiny25-attiny45-attiny85_datasheet.pdf" H 4150 3950 50  0001 C CNN
 	1    4150 3950
@@
 F 0 "P1" H 900 900 50  0000 C CNN
 F 1 "Power Connector" V 1000 1050 50  0000 C CNN
-F 2 "Terminal_Blocks:TerminalBlock_bornier-2_P5.08mm" H 900 1100 50  0001 C CNN
+F 2 "TerminalBlock:TerminalBlock_bornier-2_P5.08mm" H 900 1100 50  0001 C CNN
 F 3 "~" H 900 1100 50  0001 C CNN
 	1    900  1100
@@
 F 0 "P2" H 6250 2500 50  0000 C CNN
 F 1 "Serial Out" V 6350 2650 50  0000 C CNN
-F 2 "Pin_Headers:Pin_Header_Straight_1x02_Pitch2.54mm" H 6250 2700 50  0001 C CNN
+F 2 "Connector_PinHeader_2.54mm:PinHeader_1x02_P2.54mm_Vertical" H 6250 2700 50  0001 C CNN
 F 3 "~" H 6250 2700 50  0001 C CNN
 	1    6250 2700
@@
 F 0 "SW2" H 4400 2800 50  0000 C CNN
 F 1 "RESCUE_MODE" H 4500 2550 50  0000 C CNN
-F 2 "Buttons_Switches_ThroughHole:SW_PUSH_6mm" H 4500 2850 50  0001 C CNN
+F 2 "Button_Switch_THT:SW_PUSH_6mm" H 4500 2850 50  0001 C CNN
 F 3 "~" H 4500 2850 50  0001 C CNN
 	1    4500 2650
@@
 F 0 "SW1" H 6700 2150 50  0000 C CNN
 F 1 "RESET" H 6800 1900 50  0000 C CNN
-F 2 "Buttons_Switches_ThroughHole:SW_PUSH_6mm" H 6800 2200 50  0001 C CNN
+F 2 "Button_Switch_THT:SW_PUSH_6mm" H 6800 2200 50  0001 C CNN
 F 3 "~" H 6800 2200 50  0001 C CNN
 	1    6800 2000
